File: MotorDriver/MotorDriver KiCAD/MotorDriver KiCAD.kicad_sch (KiCad schematic)
At the start: 0 parts

Commit message: update
Other:
- company: (none) -> ${Company Name}
- title: (none) -> ${Project Title}
Changed lines of the file:
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@@
 	(generator_version "9.0")
 	(paper "A4")
+	(title_block
+		(title "${Project Title}")
+		(date "2025-07-26")
+		(rev "${Revision}")
+		(company "${Company Name}")
+		(comment 1 "${Designed By}")
+	)
 	(sheet_instances
 		(path "/"
