File: BackButtons/BackButtons KiCAD/BackButtons KiCAD.kicad_pcb (KiCad board)
At the start: 2 copper layers, 0 parts

Commit message: text vars need fixed
Other:
- board text added: "${COMMENT1} © ${COMPANY} - ${Website}"
- board text added: "${TITLE} Rev: ${REVISION}"
Changed lines of the file:
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@@
 	(paper "A4")
 	(title_block
+		(title "${Project Title}")
 		(date "2025-07-26")
+		(rev "${Revision}")
+		(company "${Company Name}")
+		(comment 1 "${Designed By}")
 	)
 	(layers
@@
 		(43 "User.3" user)
 		(45 "User.4" user)
+		(47 "User.5" user)
+		(49 "User.6" user)
+		(51 "User.7" user)
+		(53 "User.8" user)
+		(55 "User.9" user)
 	)
 	(setup
@@
 		)
 	)
+	(property "Company Name" "Philip McGaw.")
+	(property "Designed By" "Designed by Philip McGaw - philip@mcgaw.eu")
+	(property "Project Title" "Project Title")
+	(property "Revision" "0.1")
+	(property "Website" "https://philipmcgaw.com")
 	(net 0 "")
+	(gr_text "${COMMENT1}\n© ${COMPANY} - ${Website}"
+		(at 117.475 145.415 0)
+		(layer "F.SilkS")
+		(effects
+			(font
+				(size 1 1)
+				(thickness 0.15)
+			)
+		)
+	)
+	(gr_text "${TITLE}\nRev: ${REVISION}"
+		(at 117.475 139.7 0)
+		(layer "F.SilkS")
+		(effects
+			(font
+				(size 1.5 1.5)
+				(thickness 0.3)
+				(bold yes)
+			)
+		)
+	)
 	(embedded_fonts no)
 	(embedded_files
