File: BCM/KiCAD/BCM.kicad_pcb (KiCad board)
At the start: 2 copper layers, 0 parts

Commit message: updates
Parts:
- added J10: Back_9, Connector_JST:JST_XA_B04B-XASK-1_1x04_P2.50mm_Vertical, B.Cu at (137.3, 98.4)
- added J11: Back_10, Connector_JST:JST_XA_B04B-XASK-1_1x04_P2.50mm_Vertical, B.Cu at (137.3, 108.6)
- added J12: Back_11, Connector_JST:JST_XA_B04B-XASK-1_1x04_P2.50mm_Vertical, B.Cu at (137.3, 118.7)
- added J13: Back_12, Connector_JST:JST_XA_B04B-XASK-1_1x04_P2.50mm_Vertical, B.Cu at (137.3, 128.9)
- added J2: Back_1, Connector_JST:JST_XA_B04B-XASK-1_1x04_P2.50mm_Vertical, B.Cu at (96.6, 98.4)
- added J3: Back_2, Connector_JST:JST_XA_B04B-XASK-1_1x04_P2.50mm_Vertical, B.Cu at (96.6, 108.6)
- added J4: Back_3, Connector_JST:JST_XA_B04B-XASK-1_1x04_P2.50mm_Vertical, B.Cu at (96.6, 118.7)
- added J5: Back_4, Connector_JST:JST_XA_B04B-XASK-1_1x04_P2.50mm_Vertical, B.Cu at (96.6, 128.9)
- added J6: Back_5, Connector_JST:JST_XA_B04B-XASK-1_1x04_P2.50mm_Vertical, B.Cu at (117.0, 98.4)
- added J7: Back_6, Connector_JST:JST_XA_B04B-XASK-1_1x04_P2.50mm_Vertical, B.Cu at (117.0, 108.6)
- added J8: Back_7, Connector_JST:JST_XA_B04B-XASK-1_1x04_P2.50mm_Vertical, B.Cu at (117.0, 118.7)
- added J9: Back_8, Connector_JST:JST_XA_B04B-XASK-1_1x04_P2.50mm_Vertical, B.Cu at (117.0, 128.9)
- added Q1: 2N7002, Package_TO_SOT_SMD:SOT-23, F.Cu at (100.3, 94.0)
- added Q10: 2N7002, Package_TO_SOT_SMD:SOT-23, F.Cu at (141.0, 104.1)
- added Q11: 2N7002, Package_TO_SOT_SMD:SOT-23, F.Cu at (141.0, 114.3)
- added Q12: 2N7002, Package_TO_SOT_SMD:SOT-23, F.Cu at (141.0, 124.5)
- added Q2: 2N7002, Package_TO_SOT_SMD:SOT-23, F.Cu at (100.3, 103.5)
- added Q3: 2N7002, Package_TO_SOT_SMD:SOT-23, F.Cu at (100.3, 113.7)
- added Q4: 2N7002, Package_TO_SOT_SMD:SOT-23, F.Cu at (100.3, 123.8)
- added Q5: 2N7002, Package_TO_SOT_SMD:SOT-23, F.Cu at (120.7, 94.0)
- added Q6: 2N7002, Package_TO_SOT_SMD:SOT-23, F.Cu at (120.7, 104.1)
- added Q7: 2N7002, Package_TO_SOT_SMD:SOT-23, F.Cu at (120.7, 113.7)
- added Q8: 2N7002, Package_TO_SOT_SMD:SOT-23, F.Cu at (120.7, 123.8)
- added Q9: 2N7002, Package_TO_SOT_SMD:SOT-23, F.Cu at (141.0, 94.0)
- added R1: 10k, Resistor_SMD:R_0805_2012Metric_Pad1.20x1.40mm_HandSolder, F.Cu at (105.4, 94.0)
- added R10: 10k, Resistor_SMD:R_0805_2012Metric_Pad1.20x1.40mm_HandSolder, F.Cu at (155.9, 116.7)
- added R11: 330, Resistor_SMD:R_0805_2012Metric_Pad1.20x1.40mm_HandSolder, F.Cu at (155.9, 119.6)
- added R12: 330, Resistor_SMD:R_0805_2012Metric_Pad1.20x1.40mm_HandSolder, F.Cu at (155.9, 122.6)
- added R13: 10k, Resistor_SMD:R_0805_2012Metric_Pad1.20x1.40mm_HandSolder, F.Cu at (155.9, 125.5)
- added R14: 10k, Resistor_SMD:R_0805_2012Metric_Pad1.20x1.40mm_HandSolder, F.Cu at (160.6, 101.9)
- added R15: 330, Resistor_SMD:R_0805_2012Metric_Pad1.20x1.40mm_HandSolder, F.Cu at (160.6, 104.9)
- added R16: 330, Resistor_SMD:R_0805_2012Metric_Pad1.20x1.40mm_HandSolder, F.Cu at (160.6, 107.8)
- added R17: 10k, Resistor_SMD:R_0805_2012Metric_Pad1.20x1.40mm_HandSolder, F.Cu at (160.6, 110.8)
- added R18: 10k, Resistor_SMD:R_0805_2012Metric_Pad1.20x1.40mm_HandSolder, F.Cu at (160.6, 113.7)
- added R19: 10k, Resistor_SMD:R_0805_2012Metric_Pad1.20x1.40mm_HandSolder, F.Cu at (160.6, 116.7)
- added R2: 10k, Resistor_SMD:R_0805_2012Metric_Pad1.20x1.40mm_HandSolder, F.Cu at (97.2, 94.0)
- added R20: 10k, Resistor_SMD:R_0805_2012Metric_Pad1.20x1.40mm_HandSolder, F.Cu at (160.6, 119.6)
- added R21: 330, Resistor_SMD:R_0805_2012Metric_Pad1.20x1.40mm_HandSolder, F.Cu at (160.6, 122.6)
- added R22: 330, Resistor_SMD:R_0805_2012Metric_Pad1.20x1.40mm_HandSolder, F.Cu at (160.6, 125.5)
- added R23: 330, Resistor_SMD:R_0805_2012Metric_Pad1.20x1.40mm_HandSolder, F.Cu at (165.4, 101.9)
- added R24: 330, Resistor_SMD:R_0805_2012Metric_Pad1.20x1.40mm_HandSolder, F.Cu at (165.4, 104.9)
- added R25: 10k, Resistor_SMD:R_0805_2012Metric_Pad1.20x1.40mm_HandSolder, F.Cu at (165.4, 107.8)
- added R26: 10k, Resistor_SMD:R_0805_2012Metric_Pad1.20x1.40mm_HandSolder, F.Cu at (165.4, 110.8)
- added R27: 10k, Resistor_SMD:R_0805_2012Metric_Pad1.20x1.40mm_HandSolder, F.Cu at (165.4, 113.7)
- added R28: 10k, Resistor_SMD:R_0805_2012Metric_Pad1.20x1.40mm_HandSolder, F.Cu at (165.4, 116.7)
- added R29: 330, Resistor_SMD:R_0805_2012Metric_Pad1.20x1.40mm_HandSolder, F.Cu at (165.4, 119.6)
- added R3: 330, Resistor_SMD:R_0805_2012Metric_Pad1.20x1.40mm_HandSolder, F.Cu at (103.5, 94.0)
- added R30: 330, Resistor_SMD:R_0805_2012Metric_Pad1.20x1.40mm_HandSolder, F.Cu at (165.4, 122.6)
- added R31: 330, Resistor_SMD:R_0805_2012Metric_Pad1.20x1.40mm_HandSolder, F.Cu at (165.4, 125.5)
- added R32: 330, Resistor_SMD:R_0805_2012Metric_Pad1.20x1.40mm_HandSolder, F.Cu at (170.1, 101.9)
- added R33: 10k, Resistor_SMD:R_0805_2012Metric_Pad1.20x1.40mm_HandSolder, F.Cu at (170.1, 104.9)
- added R34: 10k, Resistor_SMD:R_0805_2012Metric_Pad1.20x1.40mm_HandSolder, F.Cu at (170.1, 107.8)
- added R35: 10k, Resistor_SMD:R_0805_2012Metric_Pad1.20x1.40mm_HandSolder, F.Cu at (170.1, 110.8)
- added R36: 10k, Resistor_SMD:R_0805_2012Metric_Pad1.20x1.40mm_HandSolder, F.Cu at (170.1, 113.7)
- added R37: 330, Resistor_SMD:R_0805_2012Metric_Pad1.20x1.40mm_HandSolder, F.Cu at (170.1, 116.7)
- added R38: 330, Resistor_SMD:R_0805_2012Metric_Pad1.20x1.40mm_HandSolder, F.Cu at (170.1, 119.6)
- added R39: 330, Resistor_SMD:R_0805_2012Metric_Pad1.20x1.40mm_HandSolder, F.Cu at (170.1, 122.6)
- added R4: 330, Resistor_SMD:R_0805_2012Metric_Pad1.20x1.40mm_HandSolder, F.Cu at (95.2, 94.0)
- added R40: 330, Resistor_SMD:R_0805_2012Metric_Pad1.20x1.40mm_HandSolder, F.Cu at (170.1, 125.5)
- added R41: 10k, Resistor_SMD:R_0805_2012Metric_Pad1.20x1.40mm_HandSolder, F.Cu at (174.9, 101.9)
- added R42: 10k, Resistor_SMD:R_0805_2012Metric_Pad1.20x1.40mm_HandSolder, F.Cu at (174.9, 104.9)
- added R43: 10k, Resistor_SMD:R_0805_2012Metric_Pad1.20x1.40mm_HandSolder, F.Cu at (174.9, 107.8)
- added R44: 10k, Resistor_SMD:R_0805_2012Metric_Pad1.20x1.40mm_HandSolder, F.Cu at (174.9, 110.8)
- added R45: 330, Resistor_SMD:R_0805_2012Metric_Pad1.20x1.40mm_HandSolder, F.Cu at (174.9, 113.7)
- added R46: 330, Resistor_SMD:R_0805_2012Metric_Pad1.20x1.40mm_HandSolder, F.Cu at (174.9, 116.7)
- added R47: 330, Resistor_SMD:R_0805_2012Metric_Pad1.20x1.40mm_HandSolder, F.Cu at (174.9, 119.6)
- added R48: 330, Resistor_SMD:R_0805_2012Metric_Pad1.20x1.40mm_HandSolder, F.Cu at (174.9, 122.6)
- added R5: 10k, Resistor_SMD:R_0805_2012Metric_Pad1.20x1.40mm_HandSolder, F.Cu at (155.9, 101.9)
- added R6: 330, Resistor_SMD:R_0805_2012Metric_Pad1.20x1.40mm_HandSolder, F.Cu at (155.9, 104.9)
- added R7: 10k, Resistor_SMD:R_0805_2012Metric_Pad1.20x1.40mm_HandSolder, F.Cu at (155.9, 107.8)
- added R8: 330, Resistor_SMD:R_0805_2012Metric_Pad1.20x1.40mm_HandSolder, F.Cu at (155.9, 110.8)
- added R9: 10k, Resistor_SMD:R_0805_2012Metric_Pad1.20x1.40mm_HandSolder, F.Cu at (155.9, 113.7)
- added XA1: Arduino_Mega2560_Shield, Arduino:Arduino_Mega2560_Shield, F.Cu at (61.0, 76.1)
Routing:
- net /Back Button Connectors/BackButton1: track 0.00 -> 6.24 mm
- net GND: track 0.00 -> 6.17 mm, vias 0 -> 2
- net Net-(J3-Pin_3): track 0.00 -> 4.69 mm
- net Net-(J5-Pin_3): track 0.00 -> 4.69 mm
- net Net-(J9-Pin_3): track 0.00 -> 4.69 mm
- net Net-(J8-Pin_3): track 0.00 -> 4.69 mm
- net Net-(J4-Pin_3): track 0.00 -> 4.67 mm
- net Net-(J10-Pin_3): track 0.00 -> 4.05 mm
- net Net-(J7-Pin_3): track 0.00 -> 4.05 mm
- net Net-(J6-Pin_3): track 0.00 -> 4.05 mm
- net Net-(J2-Pin_3): track 0.00 -> 4.03 mm
- net Net-(J2-Pin_1): track 0.00 -> 4.00 mm
- net /Back Button Connectors/BackLED1: track 0.00 -> 2.79 mm
- net +5V: track 0.00 -> 2.79 mm
- net Net-(Q1-G): track 0.00 -> 2.25 mm
- added copper zone on F.Cu, net +5V
- added copper zone on B.Cu, net GND
