File: BCM/KiCAD/BCM.kicad_pcb (KiCad board)
At the start: 2 copper layers, 73 parts, among them J10 Back_9, J11 Back_10, J12 Back_11, J13 Back_12, J2 Back_1, J3 Back_2, J4 Back_3, J5 Back_4, J6 Back_5, J7 Back_6, J8 Back_7, J9 Back_8, Q1 2N7002, Q10 2N7002, Q11 2N7002, Q12 2N7002, Q2 2N7002, Q3 2N7002, Q4 2N7002, Q5 2N7002, Q6 2N7002, Q7 2N7002, Q8 2N7002, Q9 2N7002

Commit message: updates
Parts:
- added J14: Eye1, Connector_JST:JST_XA_B02B-XASK-1_1x02_P2.50mm_Vertical, B.Cu at (148.0, 124.5)
- added J15: Eye2, Connector_JST:JST_XA_B02B-XASK-1_1x02_P2.50mm_Vertical, B.Cu at (158.1, 124.5)
- added J16: Nose, Connector_JST:JST_XA_B02B-XASK-1_1x02_P2.50mm_Vertical, B.Cu at (168.3, 124.5)
- added J17: S1, Connector_JST:JST_XA_B02B-XASK-1_1x02_P2.50mm_Vertical, B.Cu at (178.5, 124.5)
- added J18: S2, Connector_JST:JST_XA_B02B-XASK-1_1x02_P2.50mm_Vertical, B.Cu at (148.0, 114.3)
- added J19: S3, Connector_JST:JST_XA_B02B-XASK-1_1x02_P2.50mm_Vertical, B.Cu at (158.1, 114.3)
- added J20: S4, Connector_JST:JST_XA_B02B-XASK-1_1x02_P2.50mm_Vertical, B.Cu at (168.3, 114.3)
- added J21: S5, Connector_JST:JST_XA_B02B-XASK-1_1x02_P2.50mm_Vertical, B.Cu at (178.5, 114.3)
- added Q13: 2N7002, Package_TO_SOT_SMD:SOT-23, F.Cu at (149.2, 120.0)
- added Q14: 2N7002, Package_TO_SOT_SMD:SOT-23, F.Cu at (159.4, 120.0)
- added Q15: 2N7002, Package_TO_SOT_SMD:SOT-23, F.Cu at (169.5, 120.0)
- added Q16: 2N7002, Package_TO_SOT_SMD:SOT-23, F.Cu at (179.7, 120.0)
- added Q17: 2N7002, Package_TO_SOT_SMD:SOT-23, F.Cu at (149.2, 109.9)
- added Q18: 2N7002, Package_TO_SOT_SMD:SOT-23, F.Cu at (269.9, 103.1)
- added Q19: 2N7002, Package_TO_SOT_SMD:SOT-23, F.Cu at (269.9, 107.7)
- added Q20: 2N7002, Package_TO_SOT_SMD:SOT-23, F.Cu at (269.9, 112.4)
- added R49: 10k, Resistor_SMD:R_0805_2012Metric_Pad1.20x1.40mm_HandSolder, F.Cu at (154.3, 120.0)
- added R50: 330, Resistor_SMD:R_0805_2012Metric_Pad1.20x1.40mm_HandSolder, F.Cu at (152.4, 120.0)
- added R51: 10k, Resistor_SMD:R_0805_2012Metric_Pad1.20x1.40mm_HandSolder, F.Cu at (164.5, 120.0)
- added R52: 330, Resistor_SMD:R_0805_2012Metric_Pad1.20x1.40mm_HandSolder, F.Cu at (146.1, 120.0)
- added R53: 330, Resistor_SMD:R_0805_2012Metric_Pad1.20x1.40mm_HandSolder, F.Cu at (162.6, 120.0)
- added R54: 330, Resistor_SMD:R_0805_2012Metric_Pad1.20x1.40mm_HandSolder, F.Cu at (156.2, 120.0)
- added R55: 10k, Resistor_SMD:R_0805_2012Metric_Pad1.20x1.40mm_HandSolder, F.Cu at (174.6, 120.0)
- added R56: 330, Resistor_SMD:R_0805_2012Metric_Pad1.20x1.40mm_HandSolder, F.Cu at (172.7, 120.0)
- added R57: 330, Resistor_SMD:R_0805_2012Metric_Pad1.20x1.40mm_HandSolder, F.Cu at (166.4, 120.0)
- added R58: 10k, Resistor_SMD:R_0805_2012Metric_Pad1.20x1.40mm_HandSolder, F.Cu at (184.8, 120.0)
- added R59: 330, Resistor_SMD:R_0805_2012Metric_Pad1.20x1.40mm_HandSolder, F.Cu at (182.9, 120.0)
- added R60: 330, Resistor_SMD:R_0805_2012Metric_Pad1.20x1.40mm_HandSolder, F.Cu at (176.5, 120.0)
- added R61: 10k, Resistor_SMD:R_0805_2012Metric_Pad1.20x1.40mm_HandSolder, F.Cu at (154.3, 109.9)
- added R62: 10k, Resistor_SMD:R_0805_2012Metric_Pad1.20x1.40mm_HandSolder, F.Cu at (269.8, 127.9)
- added R63: 10k, Resistor_SMD:R_0805_2012Metric_Pad1.20x1.40mm_HandSolder, F.Cu at (269.8, 130.8)
- added R64: 10k, Resistor_SMD:R_0805_2012Metric_Pad1.20x1.40mm_HandSolder, F.Cu at (274.6, 116.1)
- added R65: 330, Resistor_SMD:R_0805_2012Metric_Pad1.20x1.40mm_HandSolder, F.Cu at (152.4, 109.9)
- added R66: 330, Resistor_SMD:R_0805_2012Metric_Pad1.20x1.40mm_HandSolder, F.Cu at (274.6, 122.0)
- added R67: 330, Resistor_SMD:R_0805_2012Metric_Pad1.20x1.40mm_HandSolder, F.Cu at (274.6, 124.9)
- added R68: 330, Resistor_SMD:R_0805_2012Metric_Pad1.20x1.40mm_HandSolder, F.Cu at (274.6, 127.9)
- added R69: 330, Resistor_SMD:R_0805_2012Metric_Pad1.20x1.40mm_HandSolder, F.Cu at (146.1, 109.9)
- added R70: 330, Resistor_SMD:R_0805_2012Metric_Pad1.20x1.40mm_HandSolder, F.Cu at (279.3, 116.1)
- added R71: 330, Resistor_SMD:R_0805_2012Metric_Pad1.20x1.40mm_HandSolder, F.Cu at (279.3, 119.0)
- added R72: 330, Resistor_SMD:R_0805_2012Metric_Pad1.20x1.40mm_HandSolder, F.Cu at (279.3, 122.0)
- moved XA1 140.5 mm to (194.3, 31.8), turned to 180 degrees
- moved R16 64.0 mm to (97.8, 120.0), turned to 90 degrees
- moved R14 63.6 mm to (99.7, 120.0), turned to 90 degrees
- moved R15 63.1 mm to (97.8, 109.9), turned to 90 degrees
- moved R29 61.5 mm to (111.8, 89.5), turned to 90 degrees
- moved R32 61.1 mm to (111.8, 120.0), turned to 90 degrees
- moved R8 59.1 mm to (97.8, 99.7), turned to 90 degrees
- moved R13 58.3 mm to (99.7, 109.9), turned to 90 degrees
- moved R30 58.3 mm to (111.8, 99.7), turned to 90 degrees
- moved R7 56.8 mm to (99.7, 99.7), turned to 90 degrees
- moved R31 55.9 mm to (111.8, 109.9), turned to 90 degrees
- moved R25 54.8 mm to (113.7, 89.5), turned to 90 degrees
- moved R45 54.8 mm to (125.7, 89.5), turned to 90 degrees
- moved R26 52.9 mm to (113.7, 99.7), turned to 90 degrees
- moved R21 52.4 mm to (120.0, 89.5), turned to 90 degrees
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Connections:
- XA1 pad D10: /Shrimp/LeftMotorDir -> unconnected-(XA1-PadD10)
- XA1 pad D11: /Shrimp/LeftMotorPWM -> unconnected-(XA1-PadD11)
- XA1 pad D12: /Shrimp/RightMotorDir -> unconnected-(XA1-PadD12)
- XA1 pad D13: /Shrimp/RightMotorPWM -> unconnected-(XA1-PadD13)
- XA1 pad D14: unconnected-(XA1-D14_TX3-PadD14) -> /Back Button Connectors/BackButton4
- XA1 pad D15: unconnected-(XA1-D15_RX3-PadD15) -> /Back Button Connectors/BackButton11
- XA1 pad D16: unconnected-(XA1-D16_TX2-PadD16) -> /Back Button Connectors/BackButton10
- XA1 pad D17: unconnected-(XA1-D17_RX2-PadD17) -> /Back Button Connectors/BackButton9
- XA1 pad D18: unconnected-(XA1-D18_TX1-PadD18) -> /Back Button Connectors/BackButton7
- XA1 pad D19: unconnected-(XA1-D19_RX1-PadD19) -> /Back Button Connectors/BackButton6
- XA1 pad D2: /Shrimp/TailServo1 -> /Back Button Connectors/BackButton12
- XA1 pad D20: unconnected-(XA1-D20_SDA-PadD20) -> /Back Button Connectors/BackButton5
- XA1 pad D21: unconnected-(XA1-D21_SCL-PadD21) -> /Back Button Connectors/BackButton3
- XA1 pad D22: unconnected-(XA1-PadD22) -> /Back Button Connectors/BackLED1
- XA1 pad D23: /Shrimp/EyesLight1 -> /Back Button Connectors/BackButton1
- XA1 pad D24: /Shrimp/EyesLight2 -> /Back Button Connectors/BackLED2
- XA1 pad D25: /Shrimp/NoseLight -> /Back Button Connectors/BackButton2
- XA1 pad D26: unconnected-(XA1-PadD26) -> /Back Button Connectors/BackLED5
- XA1 pad D27: /Shrimp/DoorBut1 -> /Back Button Connectors/BackLED3
- XA1 pad D28: /Shrimp/DoorBut2 -> /Back Button Connectors/BackLED7
- XA1 pad D29: unconnected-(XA1-PadD29) -> /Back Button Connectors/BackLED6
- XA1 pad D3: /Shrimp/TailServo2 -> /Back Button Connectors/BackLED12
- XA1 pad D30: /Back Button Connectors/BackButton1 -> /Back Button Connectors/BackLED10
- XA1 pad D31: /Back Button Connectors/BackLED1 -> /Back Button Connectors/BackLED9
- XA1 pad D32: /Back Button Connectors/BackButton2 -> /Back Button Connectors/BackLED4
- XA1 pad D33: /Back Button Connectors/BackLED2 -> /Back Button Connectors/BackLED11
- XA1 pad D34: /Back Button Connectors/BackButton3 -> /Back Button Connectors/BackLED8
- XA1 pad D35: /Back Button Connectors/BackLED3 -> /Back Button Connectors/BackButton8
- XA1 pad D36: /Back Button Connectors/BackButton4 -> unconnected-(XA1-PadD36)
- XA1 pad D37: /Back Button Connectors/BackLED4 -> unconnected-(XA1-PadD37)
- XA1 pad D38: /Back Button Connectors/BackButton5 -> unconnected-(XA1-PadD38)
- XA1 pad D39: /Back Button Connectors/BackLED5 -> unconnected-(XA1-PadD39)
- XA1 pad D4: /Shrimp/NeckServo -> unconnected-(XA1-PadD4)
- XA1 pad D40: /Back Button Connectors/BackButton6 -> unconnected-(XA1-PadD40)
- XA1 pad D41: /Back Button Connectors/BackLED6 -> unconnected-(XA1-PadD41)
- XA1 pad D42: /Back Button Connectors/BackButton7 -> unconnected-(XA1-PadD42)
- XA1 pad D43: /Back Button Connectors/BackLED7 -> unconnected-(XA1-PadD43)
- XA1 pad D44: /Back Button Connectors/BackButton8 -> unconnected-(XA1-PadD44)
- XA1 pad D45: /Back Button Connectors/BackLED8 -> unconnected-(XA1-PadD45)
- XA1 pad D46: /Back Button Connectors/BackButton9 -> /Misc Lights/SpaireLight5
- XA1 pad D47: /Back Button Connectors/BackLED9 -> /Misc Lights/SpaireLight4
- XA1 pad D48: /Back Button Connectors/BackButton10 -> /Misc Lights/SpaireLight3
- XA1 pad D49: /Back Button Connectors/BackLED10 -> /Misc Lights/SpaireLight2
- XA1 pad D5: /Shrimp/EarServo1 -> unconnected-(XA1-PadD5)
- XA1 pad D50: /Back Button Connectors/BackButton11 -> /Misc Lights/SpaireLight1
- XA1 pad D51: /Back Button Connectors/BackLED11 -> /Misc Lights/NoseLight
- XA1 pad D52: /Back Button Connectors/BackButton12 -> /Misc Lights/EyesLight2
- XA1 pad D53: /Back Button Connectors/BackLED12 -> /Misc Lights/EyesLight1
- XA1 pad D6: /Shrimp/EarServo2 -> unconnected-(XA1-PadD6)
- XA1 pad D7: /Shrimp/NoseServo1 -> unconnected-(XA1-PadD7)
- XA1 pad D8: /Shrimp/NoseServo2 -> unconnected-(XA1-PadD8)
Routing:
- net +5V: track 2.79 -> 213.7 mm, vias 0 -> 17
- net /Back Button Connectors/BackButton8: track 0.00 -> 111.7 mm
- net /Back Button Connectors/BackLED4: track 0.00 -> 109.6 mm
- net /Back Button Connectors/BackLED8: track 0.00 -> 99.4 mm
- net /Back Button Connectors/BackButton4: track 0.00 -> 88.1 mm
- net /Back Button Connectors/BackLED11: track 0.00 -> 75.6 mm
- net GND: track 6.17 -> 74.1 mm, vias 2 -> 25
- net /Back Button Connectors/BackLED10: track 0.00 -> 60.0 mm
- net /Back Button Connectors/BackLED7: track 0.00 -> 55.9 mm
- net /Back Button Connectors/BackButton12: track 0.00 -> 54.5 mm
- net /Back Button Connectors/BackButton11: track 0.00 -> 53.3 mm
- net /Back Button Connectors/BackLED9: track 0.00 -> 49.4 mm
- net /Back Button Connectors/BackLED6: track 0.00 -> 46.8 mm
- net /Back Button Connectors/BackLED3: track 0.00 -> 45.4 mm
- net /Back Button Connectors/BackButton7: track 0.00 -> 45.0 mm
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- removed copper zone on F.Cu, net +5V
Other:
- board outline added: 99.1 x 99.1 mm

Commit message: updates
Parts:
- moved R70 115.7 mm to (163.8, 109.9), turned to 90 degrees
- moved R71 105.7 mm to (174.0, 109.9), turned to 90 degrees
- moved R66 105.1 mm to (170.2, 109.9), turned to 90 degrees
- moved Q18 103.1 mm to (167.0, 109.9), turned to -90 degrees
- moved R62 99.4 mm to (172.1, 109.9), turned to -90 degrees
- moved R72 95.9 mm to (184.2, 109.9), turned to 90 degrees
- moved R67 95.4 mm to (180.4, 109.9), turned to 90 degrees
- moved Q19 92.8 mm to (177.2, 109.9), turned to -90 degrees
- moved R63 90.0 mm to (182.3, 109.9), turned to -90 degrees
- moved R68 86.0 mm to (190.5, 109.9), turned to 90 degrees
- moved Q20 82.6 mm to (187.3, 109.9), turned to -90 degrees
- moved R64 82.4 mm to (192.4, 109.9), turned to -90 degrees
- moved J16 7.64 mm to (175.9, 124.5)
- moved J20 7.64 mm to (175.9, 114.3)
- moved Q13 7.64 mm to (156.9, 120.0)
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Connections:
- XA1 pad D36: unconnected-(XA1-PadD36) -> /Misc Lights/NoseLight
- XA1 pad D37: unconnected-(XA1-PadD37) -> /Misc Lights/EyesLight1
- XA1 pad D38: unconnected-(XA1-PadD38) -> /Misc Lights/SpaireLight4
- XA1 pad D39: unconnected-(XA1-PadD39) -> /Misc Lights/SpaireLight2
- XA1 pad D4: unconnected-(XA1-PadD4) -> /Misc Lights/EyesLight2
- XA1 pad D46: /Misc Lights/SpaireLight5 -> unconnected-(XA1-PadD46)
- XA1 pad D47: /Misc Lights/SpaireLight4 -> unconnected-(XA1-PadD47)
- XA1 pad D48: /Misc Lights/SpaireLight3 -> unconnected-(XA1-PadD48)
- XA1 pad D49: /Misc Lights/SpaireLight2 -> unconnected-(XA1-PadD49)
- XA1 pad D5: unconnected-(XA1-PadD5) -> /Misc Lights/SpaireLight1
- XA1 pad D50: /Misc Lights/SpaireLight1 -> unconnected-(XA1-PadD50)
- XA1 pad D51: /Misc Lights/NoseLight -> unconnected-(XA1-PadD51)
- XA1 pad D52: /Misc Lights/EyesLight2 -> unconnected-(XA1-PadD52)
- XA1 pad D53: /Misc Lights/EyesLight1 -> unconnected-(XA1-D53_SS-PadD53)
- XA1 pad D6: unconnected-(XA1-PadD6) -> /Misc Lights/SpaireLight3
- XA1 pad D7: unconnected-(XA1-PadD7) -> /Misc Lights/SpaireLight5
Routing:
- net /Misc Lights/NoseLight: track 2.69 -> 128.5 mm
- net /Misc Lights/SpaireLight4: track 0.00 -> 119.6 mm
- net /Misc Lights/SpaireLight2: track 2.69 -> 104.3 mm
- net /Misc Lights/EyesLight1: track 10.9 -> 110.0 mm
- net /Misc Lights/SpaireLight1: track 2.69 -> 86.8 mm
- net /Misc Lights/SpaireLight5: track 0.00 -> 71.5 mm
- net /Misc Lights/EyesLight2: track 2.69 -> 68.3 mm
- net /Misc Lights/SpaireLight3: track 0.00 -> 56.7 mm
- net unconnected-(XA1-PadD44): track 36.0 -> 0.00 mm
- net unconnected-(XA1-PadD45): track 44.1 -> 21.6 mm
- net unconnected-(XA1-PadD42): track 38.0 -> 18.0 mm
- net unconnected-(XA1-PadD39): track 15.2 -> 0.00 mm
- net unconnected-(XA1-PadD37): track 14.2 -> 0.00 mm
- net unconnected-(XA1-PadD38): track 12.7 -> 0.00 mm
- net unconnected-(XA1-PadD36): track 11.6 -> 0.00 mm
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
Commit message: some updates
Parts:
- added J22: Door2, Connector_JST:JST_XA_B02B-XASK-1_1x02_P2.50mm_Vertical, B.Cu at (165.8, 104.1)
- added J23: Door1, Connector_JST:JST_XA_B02B-XASK-1_1x02_P2.50mm_Vertical, B.Cu at (155.6, 104.1)
- added J24: But1, Connector_JST:JST_XA_B02B-XASK-1_1x02_P2.50mm_Vertical, B.Cu at (175.9, 104.1)
- added J25: But2, Connector_JST:JST_XA_B02B-XASK-1_1x02_P2.50mm_Vertical, B.Cu at (186.1, 104.1)
- added J26: But3, Connector_JST:JST_XA_B02B-XASK-1_1x02_P2.50mm_Vertical, B.Cu at (155.6, 94.0)
- added J27: But4, Connector_JST:JST_XA_B02B-XASK-1_1x02_P2.50mm_Vertical, B.Cu at (165.8, 94.0)
- added J28: But5, Connector_JST:JST_XA_B02B-XASK-1_1x02_P2.50mm_Vertical, B.Cu at (175.9, 94.0)
- added J29: But6, Connector_JST:JST_XA_B02B-XASK-1_1x02_P2.50mm_Vertical, B.Cu at (186.1, 94.0)
- added R73: 10k, Resistor_SMD:R_0805_2012Metric_Pad1.20x1.40mm_HandSolder, F.Cu at (165.7, 99.7)
- added R74: 10k, Resistor_SMD:R_0805_2012Metric_Pad1.20x1.40mm_HandSolder, F.Cu at (175.9, 99.7)
- added R75: 10k, Resistor_SMD:R_0805_2012Metric_Pad1.20x1.40mm_HandSolder, F.Cu at (155.6, 99.7)
- added R76: 10k, Resistor_SMD:R_0805_2012Metric_Pad1.20x1.40mm_HandSolder, F.Cu at (186.1, 99.7)
- added R77: 10k, Resistor_SMD:R_0805_2012Metric_Pad1.20x1.40mm_HandSolder, F.Cu at (155.6, 89.5)
- added R78: 10k, Resistor_SMD:R_0805_2012Metric_Pad1.20x1.40mm_HandSolder, F.Cu at (165.7, 89.5)
- added R79: 10k, Resistor_SMD:R_0805_2012Metric_Pad1.20x1.40mm_HandSolder, F.Cu at (175.9, 89.5)
- added R80: 10k, Resistor_SMD:R_0805_2012Metric_Pad1.20x1.40mm_HandSolder, F.Cu at (186.1, 89.5)
Connections:
- XA1 pad D10: unconnected-(XA1-PadD10) -> /Misc Switches/DoorBut1
- XA1 pad D11: unconnected-(XA1-PadD11) -> /Misc Switches/DoorBut2
- XA1 pad D12: unconnected-(XA1-PadD12) -> /Misc Switches/SpaireBut1
- XA1 pad D13: unconnected-(XA1-PadD13) -> /Misc Switches/SpaireBut2
- XA1 pad D14: /Back Button Connectors/BackButton4 -> /Back Button Connectors/BackLED3
- XA1 pad D15: /Back Button Connectors/BackButton11 -> /Back Button Connectors/BackLED2
- XA1 pad D16: /Back Button Connectors/BackButton10 -> /Back Button Connectors/BackLED1
- XA1 pad D17: /Back Button Connectors/BackButton9 -> unconnected-(XA1-D17_RX2-PadD17)
- XA1 pad D18: /Back Button Connectors/BackButton7 -> unconnected-(XA1-D18_TX1-PadD18)
- XA1 pad D19: /Back Button Connectors/BackButton6 -> unconnected-(XA1-D19_RX1-PadD19)
- XA1 pad D2: /Back Button Connectors/BackButton12 -> /Back Button Connectors/BackLED9
- XA1 pad D20: /Back Button Connectors/BackButton5 -> unconnected-(XA1-D20_SDA-PadD20)
- XA1 pad D21: /Back Button Connectors/BackButton3 -> unconnected-(XA1-D21_SCL-PadD21)
- XA1 pad D22: /Back Button Connectors/BackLED1 -> unconnected-(XA1-PadD22)
- XA1 pad D23: /Back Button Connectors/BackButton1 -> unconnected-(XA1-PadD23)
- XA1 pad D24: /Back Button Connectors/BackLED2 -> unconnected-(XA1-PadD24)
- XA1 pad D25: /Back Button Connectors/BackButton2 -> unconnected-(XA1-PadD25)
- XA1 pad D26: /Back Button Connectors/BackLED5 -> unconnected-(XA1-PadD26)
- XA1 pad D27: /Back Button Connectors/BackLED3 -> unconnected-(XA1-PadD27)
- XA1 pad D28: /Back Button Connectors/BackLED7 -> /Back Button Connectors/BackButton1
- XA1 pad D29: /Back Button Connectors/BackLED6 -> unconnected-(XA1-PadD29)
- XA1 pad D3: /Back Button Connectors/BackLED12 -> /Back Button Connectors/BackLED10
- XA1 pad D30: /Back Button Connectors/BackLED10 -> /Back Button Connectors/BackButton3
- XA1 pad D31: /Back Button Connectors/BackLED9 -> /Back Button Connectors/BackButton2
- XA1 pad D32: /Back Button Connectors/BackLED4 -> /Back Button Connectors/BackLED5
- XA1 pad D33: /Back Button Connectors/BackLED11 -> /Back Button Connectors/BackButton5
- XA1 pad D34: /Back Button Connectors/BackLED8 -> /Back Button Connectors/BackLED6
- XA1 pad D35: /Back Button Connectors/BackButton8 -> /Back Button Connectors/BackButton6
- XA1 pad D36: /Misc Lights/NoseLight -> /Back Button Connectors/BackLED7
- XA1 pad D37: /Misc Lights/EyesLight1 -> /Back Button Connectors/BackButton7
- XA1 pad D38: /Misc Lights/SpaireLight4 -> /Back Button Connectors/BackButton10
- XA1 pad D39: /Misc Lights/SpaireLight2 -> /Back Button Connectors/BackButton9
- XA1 pad D4: /Misc Lights/EyesLight2 -> /Back Button Connectors/BackLED11
- XA1 pad D40: unconnected-(XA1-PadD40) -> /Back Button Connectors/BackButton4
- XA1 pad D41: unconnected-(XA1-PadD41) -> /Back Button Connectors/BackButton11
- XA1 pad D42: unconnected-(XA1-PadD42) -> /Back Button Connectors/BackButton12
- XA1 pad D43: unconnected-(XA1-PadD43) -> /Back Button Connectors/BackButton8
- XA1 pad D44: unconnected-(XA1-PadD44) -> /Misc Lights/EyesLight2
- XA1 pad D45: unconnected-(XA1-PadD45) -> /Misc Lights/EyesLight1
- XA1 pad D46: unconnected-(XA1-PadD46) -> /Misc Lights/SpaireLight1
- XA1 pad D47: unconnected-(XA1-PadD47) -> /Misc Lights/NoseLight
- XA1 pad D48: unconnected-(XA1-PadD48) -> /Misc Lights/SpaireLight5
- XA1 pad D49: unconnected-(XA1-PadD49) -> /Misc Lights/SpaireLight3
- XA1 pad D5: /Misc Lights/SpaireLight1 -> /Back Button Connectors/BackLED4
- XA1 pad D50: unconnected-(XA1-PadD50) -> /Misc Switches/SpaireBut4
- XA1 pad D51: unconnected-(XA1-PadD51) -> /Misc Switches/SpaireBut3
- XA1 pad D52: unconnected-(XA1-PadD52) -> /Misc Switches/SpaireBut6
- XA1 pad D53: unconnected-(XA1-D53_SS-PadD53) -> /Misc Switches/SpaireBut5
- XA1 pad D6: /Misc Lights/SpaireLight3 -> /Back Button Connectors/BackLED8
- XA1 pad D7: /Misc Lights/SpaireLight5 -> /Back Button Connectors/BackLED12
- XA1 pad D8: unconnected-(XA1-PadD8) -> /Misc Lights/SpaireLight2
- XA1 pad D9: unconnected-(XA1-PadD9) -> /Misc Lights/SpaireLight4
Routing:
- net /Misc Switches/SpaireBut6: track 0.00 -> 111.1 mm
- net /Misc Switches/SpaireBut5: track 0.00 -> 105.4 mm
- net /Misc Switches/SpaireBut4: track 0.00 -> 94.5 mm
- net /Misc Switches/SpaireBut3: track 0.00 -> 93.5 mm
- net /Misc Lights/SpaireLight5: track 71.5 -> 140.8 mm
- net /Misc Lights/SpaireLight2: track 104.3 -> 37.7 mm
- net /Misc Lights/SpaireLight3: track 56.7 -> 120.8 mm
- net /Misc Lights/SpaireLight4: track 119.6 -> 56.8 mm
- net /Back Button Connectors/BackButton12: track 54.5 -> 114.5 mm
- net /Misc Lights/SpaireLight1: track 86.8 -> 143.8 mm
- net /Misc Lights/EyesLight2: track 68.3 -> 122.3 mm
- net /Back Button Connectors/BackButton5: track 13.6 -> 57.9 mm
- net /Back Button Connectors/BackLED11: track 75.3 -> 31.6 mm
- net /Back Button Connectors/BackButton4: track 88.1 -> 131.8 mm
- net /Back Button Connectors/BackLED8: track 98.9 -> 56.0 mm
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- added copper zone on F.Cu, net +5V
Other:
- board size 99.1 x 99.1 mm -> 150 x 99.1 mm

Commit message: updated
Parts:
- added C1: C_Small, Capacitor_SMD:C_0805_2012Metric_Pad1.18x1.45mm_HandSolder, F.Cu at (93.3, 109.9)
- added C2: C_Small, Capacitor_SMD:C_0805_2012Metric_Pad1.18x1.45mm_HandSolder, F.Cu at (188.6, 99.7)
- added C3: C_Small, Capacitor_SMD:C_0805_2012Metric_Pad1.18x1.45mm_HandSolder, F.Cu at (149.2, 120.0)
- added C4: C_Small, Capacitor_SMD:C_0805_2012Metric_Pad1.18x1.45mm_HandSolder, F.Cu at (151.1, 120.0)
- added C5: C_Small, Capacitor_SMD:C_0805_2012Metric_Pad1.18x1.45mm_HandSolder, F.Cu at (93.3, 89.5)
- added C6: C_Small, Capacitor_SMD:C_0805_2012Metric_Pad1.18x1.45mm_HandSolder, F.Cu at (93.3, 99.7)
- added C7: C_Small, Capacitor_SMD:C_0805_2012Metric_Pad1.18x1.45mm_HandSolder, F.Cu at (93.3, 120.0)
- added C8: C_Small, Capacitor_SMD:C_0805_2012Metric_Pad1.18x1.45mm_HandSolder, F.Cu at (188.6, 89.5)
Connections:
- XA1 pad D14: /Back Button Connectors/BackLED3 -> /Back Button Connectors/BackLED5
- XA1 pad D15: /Back Button Connectors/BackLED2 -> /Back Button Connectors/BackButton5
- XA1 pad D16: /Back Button Connectors/BackLED1 -> /Back Button Connectors/BackLED3
- XA1 pad D17: unconnected-(XA1-D17_RX2-PadD17) -> /Back Button Connectors/BackButton3
- XA1 pad D18: unconnected-(XA1-D18_TX1-PadD18) -> /Back Button Connectors/BackLED2
- XA1 pad D19: unconnected-(XA1-D19_RX1-PadD19) -> /Back Button Connectors/BackButton2
- XA1 pad D20: unconnected-(XA1-D20_SDA-PadD20) -> /Back Button Connectors/BackLED1
- XA1 pad D21: unconnected-(XA1-D21_SCL-PadD21) -> /Back Button Connectors/BackButton1
- XA1 pad D28: /Back Button Connectors/BackButton1 -> unconnected-(XA1-PadD28)
- XA1 pad D30: /Back Button Connectors/BackButton3 -> unconnected-(XA1-PadD30)
- XA1 pad D31: /Back Button Connectors/BackButton2 -> unconnected-(XA1-PadD31)
- XA1 pad D32: /Back Button Connectors/BackLED5 -> unconnected-(XA1-PadD32)
- XA1 pad D33: /Back Button Connectors/BackButton5 -> unconnected-(XA1-PadD33)
Routing:
- net +5V: track 226.6 -> 423.4 mm, vias 12 -> 28
- net /Back Button Connectors/BackButton2: track 69.2 -> 30.3 mm
- net /Back Button Connectors/BackButton5: track 57.9 -> 20.0 mm
- net /Back Button Connectors/BackButton1: track 53.5 -> 17.0 mm
- net /Back Button Connectors/BackButton3: track 80.3 -> 44.1 mm
- net /Back Button Connectors/BackLED5: track 45.3 -> 10.9 mm
- net GND: track 78.7 -> 88.1 mm, vias 28 -> 33
- net /Back Button Connectors/BackLED1: track 18.8 -> 9.88 mm
- net /Back Button Connectors/BackLED2: track 30.4 -> 22.8 mm
- net /Back Button Connectors/BackLED3: track 42.4 -> 39.6 mm
- net /Back Button Connectors/BackLED4: track 70.5 -> 68.6 mm
- net /Misc Switches/SpaireBut5: track 105.4 -> 103.6 mm
- net /Misc Switches/SpaireBut4: track 94.5 -> 93.0 mm
- net /Back Button Connectors/BackButton6: track 69.5 -> 68.5 mm
- net /Back Button Connectors/BackLED6: track 57.8 -> 57.0 mm
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
Commit message: updated
Parts:
- added C10: 0.1μF, Capacitor_SMD:C_0805_2012Metric_Pad1.18x1.45mm_HandSolder, F.Cu at (238.3, 92.2)
- added C11: 10nF, Capacitor_SMD:C_0805_2012Metric_Pad1.18x1.45mm_HandSolder, F.Cu at (238.3, 95.2)
- added C12: 10pF, Capacitor_SMD:C_0805_2012Metric_Pad1.18x1.45mm_HandSolder, F.Cu at (238.3, 98.2)
- added C13: 1nF, Capacitor_SMD:C_0805_2012Metric_Pad1.18x1.45mm_HandSolder, F.Cu at (238.3, 101.2)
- added C14: 0.1uF, Capacitor_SMD:C_0805_2012Metric_Pad1.18x1.45mm_HandSolder, F.Cu at (238.3, 104.2)
- added C15: 0.1uF, Capacitor_SMD:C_0805_2012Metric_Pad1.18x1.45mm_HandSolder, F.Cu at (238.3, 107.3)
- added C16: 47μF, Capacitor_SMD:CP_Elec_5x5.9, F.Cu at (231.4, 101.0)
- added C17: 47μF, Capacitor_SMD:CP_Elec_5x5.9, F.Cu at (231.4, 107.8)
- added C9: 100μF, Capacitor_SMD:CP_Elec_5x5.9, F.Cu at (231.4, 94.1)
- added D1: SS34, Diode_SMD:D_SMA_Handsoldering, F.Cu at (232.0, 113.5)
- added D2: SS34, Diode_SMD:D_SMA_Handsoldering, F.Cu at (232.0, 118.1)
- added D3: Green, Diode_SMD:D_0805_2012Metric_Pad1.15x1.40mm_HandSolder, F.Cu at (243.1, 95.8)
- added D4: SS34, Diode_SMD:D_SMA_Handsoldering, F.Cu at (218.5, 120.7)
- added F1: Fuse, Fuse:Fuse_2010_5025Metric_Pad1.52x2.65mm_HandSolder, F.Cu at (240.9, 120.0)
- added R84: 1k, Resistor_SMD:R_0805_2012Metric_Pad1.20x1.40mm_HandSolder, F.Cu at (243.0, 98.8)
- added U1: TPS54331D, Package_SO:TI_SO-PowerPAD-8_ThermalVias, F.Cu at (241.3, 114.6)
Connections:
- XA1 pad D22: unconnected-(XA1-PadD22) -> /Back Button Connectors/BackLED6
- XA1 pad D23: unconnected-(XA1-PadD23) -> /Back Button Connectors/BackButton6
- XA1 pad D24: unconnected-(XA1-PadD24) -> /Back Button Connectors/BackLED7
- XA1 pad D25: unconnected-(XA1-PadD25) -> /Back Button Connectors/BackButton7
- XA1 pad D26: unconnected-(XA1-PadD26) -> /Back Button Connectors/BackButton10
- XA1 pad D27: unconnected-(XA1-PadD27) -> /Back Button Connectors/BackButton9
- XA1 pad D28: unconnected-(XA1-PadD28) -> /Back Button Connectors/BackButton4
- XA1 pad D29: unconnected-(XA1-PadD29) -> /Back Button Connectors/BackButton11
- XA1 pad D30: unconnected-(XA1-PadD30) -> /Back Button Connectors/BackButton12
- XA1 pad D31: unconnected-(XA1-PadD31) -> /Back Button Connectors/BackButton8
- XA1 pad D32: unconnected-(XA1-PadD32) -> /Misc Lights/EyesLight2
- XA1 pad D33: unconnected-(XA1-PadD33) -> /Misc Lights/EyesLight1
- XA1 pad D34: /Back Button Connectors/BackLED6 -> /Misc Lights/SpaireLight1
- XA1 pad D35: /Back Button Connectors/BackButton6 -> /Misc Lights/NoseLight
- XA1 pad D36: /Back Button Connectors/BackLED7 -> /Misc Lights/SpaireLight5
- XA1 pad D37: /Back Button Connectors/BackButton7 -> /Misc Lights/SpaireLight3
- XA1 pad D38: /Back Button Connectors/BackButton10 -> /Misc Switches/SpaireBut4
- XA1 pad D39: /Back Button Connectors/BackButton9 -> /Misc Switches/SpaireBut3
- XA1 pad D40: /Back Button Connectors/BackButton4 -> /Misc Switches/SpaireBut6
- XA1 pad D41: /Back Button Connectors/BackButton11 -> /Misc Switches/SpaireBut5
- XA1 pad D42: /Back Button Connectors/BackButton12 -> unconnected-(XA1-PadD42)
- XA1 pad D43: /Back Button Connectors/BackButton8 -> unconnected-(XA1-PadD43)
- XA1 pad D44: /Misc Lights/EyesLight2 -> unconnected-(XA1-PadD44)
- XA1 pad D45: /Misc Lights/EyesLight1 -> unconnected-(XA1-PadD45)
- XA1 pad D46: /Misc Lights/SpaireLight1 -> unconnected-(XA1-PadD46)
- XA1 pad D47: /Misc Lights/NoseLight -> unconnected-(XA1-PadD47)
- XA1 pad D48: /Misc Lights/SpaireLight5 -> unconnected-(XA1-PadD48)
- XA1 pad D49: /Misc Lights/SpaireLight3 -> unconnected-(XA1-PadD49)
- XA1 pad D50: /Misc Switches/SpaireBut4 -> unconnected-(XA1-PadD50)
- XA1 pad D51: /Misc Switches/SpaireBut3 -> unconnected-(XA1-PadD51)
- XA1 pad D52: /Misc Switches/SpaireBut6 -> unconnected-(XA1-PadD52)
- XA1 pad D53: /Misc Switches/SpaireBut5 -> unconnected-(XA1-D53_SS-PadD53)
- XA1 pad VIN: +VDC -> unconnected-(XA1-PadVIN)
Routing:
- net /Misc Switches/SpaireBut6: track 111.1 -> 104.1 mm
- net GND: track 88.1 -> 94.9 mm
- net /Misc Switches/SpaireBut5: track 103.6 -> 97.0 mm
- net /Misc Lights/SpaireLight1: track 143.8 -> 137.3 mm
- net /Back Button Connectors/BackLED6: track 57.0 -> 50.7 mm
- net /Back Button Connectors/BackButton9: track 55.4 -> 49.1 mm
- net /Back Button Connectors/BackButton7: track 81.0 -> 74.7 mm
- net /Back Button Connectors/BackButton4: track 131.8 -> 125.5 mm
- net /Misc Switches/SpaireBut4: track 93.0 -> 86.7 mm
- net /Misc Lights/NoseLight: track 136.0 -> 129.7 mm
- net /Misc Lights/EyesLight2: track 122.3 -> 116.0 mm
- net /Misc Lights/EyesLight1: track 114.6 -> 108.3 mm
- net /Back Button Connectors/BackButton8: track 125.8 -> 119.5 mm
- net /Back Button Connectors/BackButton12: track 114.1 -> 107.8 mm
- net /Back Button Connectors/BackButton11: track 95.4 -> 89.1 mm
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