File: BCM/KiCAD/misc lights.kicad_sch (KiCad schematic)
At the start: 40 parts, among them J14 Eye1, J15 Eye2, J16 Nose, J17 S1, J18 S2, J19 S3, J20 S4, J21 S5, Q13 2N7002, Q14 2N7002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

Commit message: updated
Parts:
- added C5, C6, C7, C8: C_Small, Capacitor_SMD:C_0805_2012Metric_Pad1.18x1.45mm_HandSolder, symbol Device:C_Small
Connections:
- net +5V: now also C5.1, C6.1, C7.1, C8.1
- net GND: now also C5.2, C6.2, C7.2, C8.2
