File: BCM/KiCAD/shrimp.kicad_sch (KiCad schematic)
At the start: 1 part

Commit message: work
Parts:
- XA1: footprint (none) -> Arduino:Arduino_Mega2560_Shield
Connections:
- net +5V: now reaches XA1.5V1 (5V)
- net +5V: now also XA1.5V3 (5V), XA1.5V4 (5V)
- net EyesLight1: now reaches XA1.D10
- net EyesLight2: now reaches XA1.D11
- net NoseLight: now reaches XA1.D12
- net TailServo1: now reaches XA1.D2 (D2_INT0)
- net DoorBut1: now reaches XA1.D27
- net DoorBut2: now reaches XA1.D28
- net TailServo2: now reaches XA1.D3 (D3_INT1)
- net BackBut1: now reaches XA1.D30
- net BackBut2: now reaches XA1.D31
- net BackBut3: now reaches XA1.D32
- net BackBut4: now reaches XA1.D33
- net BackBut5: now reaches XA1.D34
- net BackBut6: now reaches XA1.D35
- net BackBut7: now reaches XA1.D36
- net BackBut8: now reaches XA1.D37
- net BackBut9: now reaches XA1.D38
- net BackBut10: now reaches XA1.D39
- net NeckServo: now reaches XA1.D4
- net BackBut11: now reaches XA1.D40
- net BackBut12: now reaches XA1.D41
- net BackLED1: now reaches XA1.D42
- net BackLED2: now reaches XA1.D43
- net BackLED3: now reaches XA1.D44
- net BackLED4: now reaches XA1.D45
- net BackLED5: now reaches XA1.D46
- net BackLED6: now reaches XA1.D47
- net BackLED7: now reaches XA1.D48
- net BackLED8: now reaches XA1.D49
- net EarServo1: now reaches XA1.D5
- net BackLED9: now reaches XA1.D50
- net BackLED10: now reaches XA1.D51
- net BackLED11: now reaches XA1.D52
- net BackLED12: now reaches XA1.D53 (D53_SS)
- net EarServo2: now reaches XA1.D6
- net NoseServo1: now reaches XA1.D7
- net NoseServo2: now reaches XA1.D8
- net GND: now reaches XA1.GND1 (GND), XA1.GND2 (GND), XA1.GND3 (GND), XA1.GND5 (GND), XA1.GND6 (GND)
- net +VDC: now reaches XA1.VIN
- no-connect marks 0 -> 2

Commit message: Update shrimp.kicad_sch
Connections:
- net EyesLight1: now also XA1.D13; no longer XA1.D10
- net EyesLight2: now also XA1.D22; no longer XA1.D11
- net NoseLight: now also XA1.D23; no longer XA1.D12
- new net LeftMotorServo: XA1.D10
- new net RightMotorServo: XA1.D11

Commit message: updates
Connections:
- net BackBut10: now also XA1.D48; no longer XA1.D39
- net BackBut11: now also XA1.D50; no longer XA1.D40
- net BackBut12: now also XA1.D52; no longer XA1.D41
- net BackBut2: now also XA1.D32; no longer XA1.D31
- net BackBut3: now also XA1.D34; no longer XA1.D32
- net BackBut4: now also XA1.D36; no longer XA1.D33
- net BackBut5: now also XA1.D38; no longer XA1.D34
- net BackBut6: now also XA1.D40; no longer XA1.D35
- net BackBut7: now also XA1.D42; no longer XA1.D36
- net BackBut8: now also XA1.D44; no longer XA1.D37
- net BackBut9: now also XA1.D46; no longer XA1.D38
- net BackLED1: now also XA1.D31; no longer XA1.D42
- net BackLED10: now also XA1.D49; no longer XA1.D51
- net BackLED11: now also XA1.D51; no longer XA1.D52
- net BackLED2: now also XA1.D33; no longer XA1.D43
- net BackLED3: now also XA1.D35; no longer XA1.D44
- net BackLED4: now also XA1.D37; no longer XA1.D45
- net BackLED5: now also XA1.D39; no longer XA1.D46
- net BackLED6: now also XA1.D41; no longer XA1.D47
- net BackLED7: now also XA1.D43; no longer XA1.D48
- net BackLED8: now also XA1.D45; no longer XA1.D49
- net BackLED9: now also XA1.D47; no longer XA1.D50
- net EyesLight1: now also XA1.D23; no longer XA1.D13
- net EyesLight2: now also XA1.D24; no longer XA1.D22
- net NoseLight: now also XA1.D25; no longer XA1.D23
- net ADC_I: now reaches XA1.A0
- net ADC_V: now reaches XA1.A1
- net RightMotorDir: now reaches XA1.D12
- net LeftMotorServo renamed LeftMotorDir
- net RightMotorServo renamed LeftMotorPWM
- new net RightMotorPWM: XA1.D13

Commit message: updates
Connections:
- net BackBut1: now also XA1.D23; no longer XA1.D30
- net BackBut10: now also XA1.D16 (D16_TX2); no longer XA1.D48
- net BackBut11: now also XA1.D15 (D15_RX3); no longer XA1.D50
- net BackBut12: now also XA1.D2 (D2_INT0); no longer XA1.D52
- net BackBut2: now also XA1.D25; no longer XA1.D32
- net BackBut3: now also XA1.D21 (D21_SCL); no longer XA1.D34
- net BackBut4: now also XA1.D14 (D14_TX3); no longer XA1.D36
- net BackBut5: now also XA1.D20 (D20_SDA); no longer XA1.D38
- net BackBut6: now also XA1.D19 (D19_RX1); no longer XA1.D40
- net BackBut7: now also XA1.D18 (D18_TX1); no longer XA1.D42
- net BackBut8: now also XA1.D35; no longer XA1.D44
- net BackBut9: now also XA1.D17 (D17_RX2); no longer XA1.D46
- net BackLED1: now also XA1.D22; no longer XA1.D31
- net BackLED10: now also XA1.D30; no longer XA1.D49
- net BackLED11: now also XA1.D33; no longer XA1.D51
- net BackLED12: now also XA1.D3 (D3_INT1); no longer XA1.D53 (D53_SS)
- net BackLED2: now also XA1.D24; no longer XA1.D33
- net BackLED3: now also XA1.D27; no longer XA1.D35
- net BackLED4: now also XA1.D32; no longer XA1.D37
- net BackLED5: now also XA1.D26; no longer XA1.D39
- net BackLED6: now also XA1.D29; no longer XA1.D41
- net BackLED7: now also XA1.D28; no longer XA1.D43
- net BackLED8: now also XA1.D34; no longer XA1.D45
- net BackLED9: now also XA1.D31; no longer XA1.D47
- net DoorBut1: no longer XA1.D27
- net DoorBut2: no longer XA1.D28
- net EarServo1: no longer XA1.D5
- net EarServo2: no longer XA1.D6
- net EyesLight1: now also XA1.D53 (D53_SS); no longer XA1.D23
- net EyesLight2: now also XA1.D52; no longer XA1.D24
- net LeftMotorDir: no longer XA1.D10
- net LeftMotorPWM: no longer XA1.D11
- net NeckServo: no longer XA1.D4
- net NoseLight: now also XA1.D51; no longer XA1.D25
- net NoseServo1: no longer XA1.D7
- net NoseServo2: no longer XA1.D8
- net RightMotorDir: no longer XA1.D12
- net RightMotorPWM: no longer XA1.D13
- net TailServo1: no longer XA1.D2 (D2_INT0)
- net TailServo2: no longer XA1.D3 (D3_INT1)
- new net SpaireLight1: XA1.D50
- new net SpaireLight2: XA1.D49
- new net SpaireLight3: XA1.D48
- new net SpaireLight4: XA1.D47
- new net SpaireLight5: XA1.D46

Commit message: updates
Connections:
- net EyesLight1: now also XA1.D37; no longer XA1.D53 (D53_SS)
- net EyesLight2: now also XA1.D4; no longer XA1.D52
- net NoseLight: now also XA1.D36; no longer XA1.D51
- net SpaireLight1: now also XA1.D5; no longer XA1.D50
- net SpaireLight2: now also XA1.D39; no longer XA1.D49
- net SpaireLight3: now also XA1.D6; no longer XA1.D48
- net SpaireLight4: now also XA1.D38; no longer XA1.D47
- net SpaireLight5: now also XA1.D7; no longer XA1.D46
Changed lines of the file:
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@@
 	(hierarchical_label "SpaireLight2"
 		(shape output)
-		(at 195.58 130.81 0)
+		(at 195.58 105.41 0)
 		(effects
 			(font
@@
 	(hierarchical_label "EyesLight1"
 		(shape output)
-		(at 195.58 140.97 0)
+		(at 195.58 100.33 0)
 		(effects
 			(font
@@
 	(hierarchical_label "NoseLight"
 		(shape output)
-		(at 195.58 135.89 0)
+		(at 195.58 97.79 0)
 		(effects
 			(font
@@
 	(hierarchical_label "SpaireLight5"
 		(shape output)
-		(at 195.58 123.19 0)
+		(at 195.58 44.45 0)
 		(effects
 			(font
@@
 	(hierarchical_label "SpaireLight3"
 		(shape output)
-		(at 195.58 128.27 0)
+		(at 195.58 41.91 0)
 		(effects
 			(font
@@
 	(hierarchical_label "SpaireLight4"
 		(shape output)
-		(at 195.58 125.73 0)
+		(at 195.58 102.87 0)
 		(effects
 			(font
@@
 	(hierarchical_label "SpaireLight1"
 		(shape output)
-		(at 195.58 133.35 0)
+		(at 195.58 39.37 0)
 		(effects
 			(font
@@
 	(hierarchical_label "EyesLight2"
 		(shape output)
-		(at 195.58 138.43 0)
-		(effects
-			(font
+		(at 195.58 36.83 0)
+		(effects
+			(font

Commit message: some updates
Connections:
- net BackBut1: now also XA1.D28; no longer XA1.D23
- net BackBut10: now also XA1.D38; no longer XA1.D16 (D16_TX2)
- net BackBut11: now also XA1.D41; no longer XA1.D15 (D15_RX3)
- net BackBut12: now also XA1.D42; no longer XA1.D2 (D2_INT0)
- net BackBut2: now also XA1.D31; no longer XA1.D25
- net BackBut3: now also XA1.D30; no longer XA1.D21 (D21_SCL)
- net BackBut4: now also XA1.D40; no longer XA1.D14 (D14_TX3)
- net BackBut5: now also XA1.D33; no longer XA1.D20 (D20_SDA)
- net BackBut6: now also XA1.D35; no longer XA1.D19 (D19_RX1)
- net BackBut7: now also XA1.D37; no longer XA1.D18 (D18_TX1)
- net BackBut8: now also XA1.D43; no longer XA1.D35
- net BackBut9: now also XA1.D39; no longer XA1.D17 (D17_RX2)
- net BackLED1: now also XA1.D16 (D16_TX2); no longer XA1.D22
- net BackLED10: now also XA1.D3 (D3_INT1); no longer XA1.D30
- net BackLED11: now also XA1.D4; no longer XA1.D33
- net BackLED12: now also XA1.D7; no longer XA1.D3 (D3_INT1)
- net BackLED2: now also XA1.D15 (D15_RX3); no longer XA1.D24
- net BackLED3: now also XA1.D14 (D14_TX3); no longer XA1.D27
- net BackLED4: now also XA1.D5; no longer XA1.D32
- net BackLED5: now also XA1.D32; no longer XA1.D26
- net BackLED6: now also XA1.D34; no longer XA1.D29
- net BackLED7: now also XA1.D36; no longer XA1.D28
- net BackLED8: now also XA1.D6; no longer XA1.D34
- net BackLED9: now also XA1.D2 (D2_INT0); no longer XA1.D31
- net DoorBut1: now also XA1.D10
- net DoorBut2: now also XA1.D11
- net EyesLight1: now also XA1.D45; no longer XA1.D37
- net EyesLight2: now also XA1.D44; no longer XA1.D4
- net NoseLight: now also XA1.D47; no longer XA1.D36
- net SpaireLight1: now also XA1.D46; no longer XA1.D5
- net SpaireLight2: now also XA1.D8; no longer XA1.D39
- net SpaireLight3: now also XA1.D49; no longer XA1.D6
- net SpaireLight4: now also XA1.D9; no longer XA1.D38
- net SpaireLight5: now also XA1.D48; no longer XA1.D7
- net SpaireBut1: now reaches XA1.D12
- net SpaireBut2: now reaches XA1.D13
- net SpaireBut4: now reaches XA1.D50
- net SpaireBut3: now reaches XA1.D51
- net SpaireBut6: now reaches XA1.D52
- net SpaireBut5: now reaches XA1.D53 (D53_SS)

Commit message: updated
Connections:
- net BackBut1: now also XA1.D21 (D21_SCL); no longer XA1.D28
- net BackBut2: now also XA1.D19 (D19_RX1); no longer XA1.D31
- net BackBut3: now also XA1.D17 (D17_RX2); no longer XA1.D30
- net BackBut5: now also XA1.D15 (D15_RX3); no longer XA1.D33
- net BackLED1: now also XA1.D20 (D20_SDA); no longer XA1.D16 (D16_TX2)
- net BackLED2: now also XA1.D18 (D18_TX1); no longer XA1.D15 (D15_RX3)
- net BackLED3: now also XA1.D16 (D16_TX2); no longer XA1.D14 (D14_TX3)
- net BackLED5: now also XA1.D14 (D14_TX3); no longer XA1.D32

Commit message: updated
Connections:
- net BackBut10: now also XA1.D26; no longer XA1.D38
- net BackBut11: now also XA1.D29; no longer XA1.D41
- net BackBut12: now also XA1.D30; no longer XA1.D42
- net BackBut4: now also XA1.D28; no longer XA1.D40
- net BackBut6: now also XA1.D23; no longer XA1.D35
- net BackBut7: now also XA1.D25; no longer XA1.D37
- net BackBut8: now also XA1.D31; no longer XA1.D43
- net BackBut9: now also XA1.D27; no longer XA1.D39
- net BackLED6: now also XA1.D22; no longer XA1.D34
- net BackLED7: now also XA1.D24; no longer XA1.D36
- net EyesLight1: now also XA1.D33; no longer XA1.D45
- net EyesLight2: now also XA1.D32; no longer XA1.D44
- net NoseLight: now also XA1.D35; no longer XA1.D47
- net SpaireBut3: now also XA1.D39; no longer XA1.D51
- net SpaireBut4: now also XA1.D38; no longer XA1.D50
- net SpaireBut5: now also XA1.D41; no longer XA1.D53 (D53_SS)
- net SpaireBut6: now also XA1.D40; no longer XA1.D52
- net SpaireLight1: now also XA1.D34; no longer XA1.D46
- net SpaireLight3: now also XA1.D37; no longer XA1.D49
- net SpaireLight5: now also XA1.D36; no longer XA1.D48
- net +VDC: no longer names the net of XA1.VIN
