File: BCM/KiCAD/shrimp.kicad_sch (KiCad schematic)
At the start: 1 part

Commit message: SDA SCL recovered
Connections:
- net BackBut1: now also XA1.D23; no longer XA1.D21 (D21_SCL)
- net BackBut10: now also XA1.D28; no longer XA1.D26
- net BackBut11: now also XA1.D31; no longer XA1.D29
- net BackBut12: now also XA1.D32; no longer XA1.D30
- net BackBut4: now also XA1.D30; no longer XA1.D28
- net BackBut6: now also XA1.D25; no longer XA1.D23
- net BackBut7: now also XA1.D27; no longer XA1.D25
- net BackBut8: now also XA1.D33; no longer XA1.D31
- net BackBut9: now also XA1.D29; no longer XA1.D27
- net BackLED1: now also XA1.D22; no longer XA1.D20 (D20_SDA)
- net BackLED6: now also XA1.D24; no longer XA1.D22
- net BackLED7: now also XA1.D26; no longer XA1.D24
- net EyesLight1: now also XA1.D35; no longer XA1.D33
- net EyesLight2: now also XA1.D34; no longer XA1.D32
- net NoseLight: now also XA1.D37; no longer XA1.D35
- net SpaireBut3: now also XA1.D41; no longer XA1.D39
- net SpaireBut4: now also XA1.D40; no longer XA1.D38
- net SpaireBut5: now also XA1.D43; no longer XA1.D41
- net SpaireBut6: now also XA1.D42; no longer XA1.D40
- net SpaireLight1: now also XA1.D36; no longer XA1.D34
- net SpaireLight3: now also XA1.D39; no longer XA1.D37
- net SpaireLight5: now also XA1.D38; no longer XA1.D36

Commit message: added servos
Connections:
- net EarServo1: now also XA1.D50
- net EarServo2: now also XA1.D51
- net NeckServo: now also XA1.D49
- net NoseServo1: now also XA1.D52
- net NoseServo2: now also XA1.D53 (D53_SS)
- net TailServo1: now also XA1.D47
- net TailServo2: now also XA1.D48
- net SpairServo1: now reaches XA1.D44
- net SpairServo2: now reaches XA1.D45
- net SpairServo3: now reaches XA1.D46
- no-connect marks 2 -> 6
Changed lines of the file:
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@@
+	)
+	(no_connect
+		(at 127 52.07)
 	)
 	(no_connect
@@
 	)
 	(no_connect
+		(at 127 59.69)
+	)
+	(no_connect
 		(at 127 34.29)
 	)
+	(no_connect
+		(at 127 57.15)
+	)
+	(no_connect
+		(at 127 54.61)
+	)
 	(wire
 		(pts
@@
 	(wire
 		(pts
-			(xy 238.76 50.8) (xy 241.3 50.8)
+			(xy 85.09 83.82) (xy 87.63 83.82)
 		)
 		(stroke
@@
 	(wire
 		(pts
-			(xy 193.04 120.65) (xy 198.12 120.65)
+			(xy 193.04 120.65) (xy 195.58 120.65)
 		)
 		(stroke
@@
 	(wire
 		(pts
-			(xy 238.76 58.42) (xy 241.3 58.42)
+			(xy 85.09 91.44) (xy 87.63 91.44)
 		)
 		(stroke
@@
 	(wire
 		(pts
-			(xy 193.04 118.11) (xy 198.12 118.11)
-		)
-		(stroke
-			(width 0)
-			(type default)
-		)
-	)
-	(wire
-		(pts
-			(xy 238.76 53.34) (xy 241.3 53.34)
+			(xy 193.04 118.11) (xy 195.58 118.11)
+		)
+		(stroke
+			(width 0)
+			(type default)
+		)
+	)
+	(wire
+		(pts
+			(xy 85.09 86.36) (xy 87.63 86.36)
 		)
 		(stroke
@@
 	(wire
 		(pts
-			(xy 238.76 55.88) (xy 241.3 55.88)
+			(xy 85.09 88.9) (xy 87.63 88.9)
 		)
 		(stroke
@@
 		)
 	)
+	(hierarchical_label "SpairServo3"
+		(shape output)
+		(at 195.58 123.19 0)
+		(effects
+			(font
+				(size 1.27 1.27)
+			)
+			(justify left)
+		)
+	)
 	(hierarchical_label "BackBut5"
 		(shape input)
@@
 		)
 	)
+	(hierarchical_label "SpairServo2"
+		(shape output)
+		(at 195.58 120.65 0)
+		(effects
+			(font
+				(size 1.27 1.27)
+			)
+			(justify left)
+		)
+	)
 	(hierarchical_label "BackLED3"
 		(shape output)
@@
 	(hierarchical_label "LeftMotorDir"
 		(shape output)
-		(at 241.3 50.8 0)
+		(at 87.63 83.82 0)
 		(effects
 			(font
@@
 		)
 	)
+	(hierarchical_label "SpairServo1"
+		(shape output)
+		(at 195.58 118.11 0)
+		(effects
+			(font
+				(size 1.27 1.27)
+			)
+			(justify left)
+		)
+	)
 	(hierarchical_label "BackLED7"
 		(shape output)
@@
 	(hierarchical_label "NeckServo"
 		(shape output)
-		(at 218.44 132.08 0)
+		(at 195.58 130.81 0)
 		(effects
 			(font
@@
 	(hierarchical_label "RightMotorDir"
 		(shape output)
-		(at 241.3 55.88 0)
+		(at 87.63 88.9 0)
 		(effects
 			(font
@@
 	(hierarchical_label "EarServo1"
 		(shape output)
-		(at 218.44 134.62 0)
+		(at 195.58 133.35 0)
 		(effects
 			(font
@@
 	(hierarchical_label "NoseServo2"
 		(shape output)
-		(at 218.44 142.24 0)
+		(at 195.58 140.97 0)
 		(effects
 			(font
@@
 	(hierarchical_label "RightMotorPWM"
 		(shape output)
-		(at 241.3 58.42 0)
+		(at 87.63 91.44 0)
 		(effects
 			(font
@@
 	(hierarchical_label "LeftMotorPWM"
 		(shape output)
-		(at 241.3 53.34 0)
+		(at 87.63 86.36 0)
 		(effects
 			(font
@@
 	(hierarchical_label "TailServo1"
 		(shape output)
-		(at 218.44 127 0)
+		(at 195.58 125.73 0)
 		(effects
 			(font
@@
 	(hierarchical_label "TailServo2"
 		(shape output)
-		(at 218.44 129.54 0)
+		(at 195.58 128.27 0)
 		(effects
 			(font
@@
 	(hierarchical_label "NoseServo1"
 		(shape output)
-		(at 218.44 139.7 0)
+		(at 195.58 138.43 0)
 		(effects
 			(font
@@
 	(hierarchical_label "EarServo2"
 		(shape output)
-		(at 218.44 137.16 0)
-		(effects
-			(font
+		(at 195.58 135.89 0)
+		(effects
+			(font
