File: BCM/KiCAD/BCM.kicad_sch (KiCad schematic)
At the start: 0 parts

Commit message: started
Other:
- added sheet Shrimp (shrimp.kicad_sch)
Changed lines of the file:
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@@
 		(comment 1 "${Designed By}")
+	)
+	(sheet
+		(at 124.46 58.42)
+		(size 49.53 66.04)
+		(exclude_from_sim no)
+		(in_bom yes)
+		(on_board yes)
+		(dnp no)
+		(fields_autoplaced yes)
+		(stroke
+			(width 0.1524)
+			(type solid)
+		)
+		(fill
+			(color 0 0 0 0.0000)
+		)
+		(property "Sheetname" "Shrimp"
+			(at 124.46 57.7084 0)
+			(effects
+				(font
+					(size 1.27 1.27)
+				)
+				(justify left bottom)
+			)
+		)
+		(property "Sheetfile" "shrimp.kicad_sch"
+			(at 124.46 125.0446 0)
+			(effects
+				(font
+					(size 1.27 1.27)
+				)
+				(justify left top)
+				(hide yes)
+			)
+		)
+		(instances
+			(project "BCM"
+				(path "/4f572b99-5eee-4690-a22b-0d608e2cc8a2"
+					(page "2")
+				)
+			)
+		)
 	)
 	(sheet_instances

Commit message: work
Parts:
- added J1: Screw_Terminal_01x06, Component Search Engine:Pluggable Terminal Blocks SDC 2,5 14-PV-5,0 0-ZB, symbol Wire to Board:Screw_Terminal_01x06
Connections:
- new net +BATT: J1.1 (Pin_1), J1.2 (Pin_2)
- new net +VDC: J1.3 (Pin_3)
- new net GND: J1.4 (Pin_4), J1.5 (Pin_5), J1.6 (Pin_6)
Other:
- sheet Shrimp ports: added BackBut1, BackBut10, BackBut11, BackBut12, BackBut2, BackBut3, BackBut4, BackBut5, BackBut6, BackBut7, BackBut8, BackBut9, BackLED1, BackLED10, BackLED11, BackLED12, BackLED2, BackLED3, BackLED4, BackLED5, BackLED6, BackLED7, BackLED8, BackLED9, DoorBut1, DoorBut2, EarServo1, EarServo2, EyesLight1, EyesLight2, NeckServo, NoseLight, NoseServo1, NoseServo2, TailServo1, TailServo2; removed none

Commit message: Update BCM.kicad_sch
Parts:
- removed J1: Screw_Terminal_01x06, Component Search Engine:Pluggable Terminal Blocks SDC 2,5 14-PV-5,0 0-ZB, symbol Wire to Board:Screw_Terminal_01x06
- added J1: Conn_01x06_Socket, symbol Connector:Conn_01x06_Socket
Connections:
- net +BATT: now also J1.1 (Pin_1), J1.2 (Pin_2)
- net +VDC: now also J1.3 (Pin_3)
- net GND: now also J1.4 (Pin_4), J1.5 (Pin_5), J1.6 (Pin_6)
Changed lines of the file:
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@@
+	)
+	(symbol
+		(lib_id "Connector:Conn_01x06_Socket")
+		(at 30.48 30.48 0)
+		(mirror y)
+		(unit 1)
+		(exclude_from_sim no)
+		(in_bom yes)
+		(on_board yes)
+		(dnp no)
+		(fields_autoplaced yes)
+		(property "Reference" "J1"
+			(at 31.115 20.32 0)
+			(effects
+				(font
+					(size 1.27 1.27)
+				)
+			)
+		)
+		(property "Value" "Conn_01x06_Socket"
+			(at 31.115 22.86 0)
+			(effects
+				(font
+					(size 1.27 1.27)
+				)
+			)
+		)
+		(property "Footprint" ""
+			(at 30.48 30.48 0)
+			(effects
+				(font
+					(size 1.27 1.27)
+				)
+				(hide yes)
+			)
+		)
+		(property "Datasheet" "~"
+			(at 30.48 30.48 0)
+			(effects
+				(font
+					(size 1.27 1.27)
+				)
+				(hide yes)
+			)
+		)
+		(property "Description" "Generic connector, single row, 01x06, script generated"
+			(at 30.48 30.48 0)
+			(effects
+				(font
+					(size 1.27 1.27)
+				)
+				(hide yes)
+			)
+		)
+		(pin "1"
+		)
+		(pin "2"
+		)
+		(pin "3"
+		)
+		(pin "4"
+		)
+		(pin "6"
+		)
+		(pin "5"
+		)
+		(instances
+			(project ""
+				(path "/4f572b99-5eee-4690-a22b-0d608e2cc8a2"
+					(reference "J1")
+					(unit 1)
+				)
+			)
+		)
 	)
 	(symbol
@@
 					(unit 1)
 				)
-			)
-		)
-	)
-	(symbol
-		(lib_id "Wire to Board:Screw_Terminal_01x06")
-		(at 30.48 30.48 0)
-		(mirror y)
-		(unit 1)
-		(exclude_from_sim no)
-		(in_bom yes)
-		(on_board yes)
-		(dnp no)
-		(fields_autoplaced yes)
-		(property "Reference" "J1"
-			(at 30.48 19.05 0)
-			(effects
-				(font
-					(size 1.27 1.27)
-				)
-			)
-		)
-		(property "Value" "Screw_Terminal_01x06"
-			(at 30.48 21.59 0)
-			(effects
-				(font
-					(size 1.27 1.27)
-				)
-			)
-		)
-		(property "Footprint" "Component Search Engine:Pluggable Terminal Blocks SDC 2,5 14-PV-5,0 0-ZB"
-			(at 30.48 30.48 0)
-			(effects
-				(font
-					(size 1.27 1.27)
-				)
-				(hide yes)
-			)
-		)
-		(property "Datasheet" "https://labbook.skippy.org.uk/projects/kicad/screw"
-			(at 30.48 30.48 0)
-			(effects
-				(font
-					(size 1.27 1.27)
-				)
-				(hide yes)
-			)
-		)
-		(property "Description" "Generic screw terminal, single row, 01x06, script generated (kicad-library-utils/schlib/autogen/connector/)"
-			(at 30.48 30.48 0)
-			(effects
-				(font
-					(size 1.27 1.27)
-				)
-				(hide yes)
-			)
-		)
-		(pin "4"
-		)
-		(pin "3"
-		)
-		(pin "1"
-		)
-		(pin "6"
-		)
-		(pin "5"
-		)
-		(pin "2"
-		)
-		(instances
-			(project ""
-				(path "/4f572b99-5eee-4690-a22b-0d608e2cc8a2"
-					(reference "J1")
-					(unit 1)
-				)

Commit message: updates
Other:
- added sheet Back Button Connectors (Back Button Connectors.kicad_sch)
- sheet Shrimp ports: added ADC_I, ADC_V, LeftMotorDir, LeftMotorPWM, RightMotorDir, RightMotorPWM; removed none

Commit message: updates
Other:
- added sheet Misc Lights (misc lights.kicad_sch)
- sheet Shrimp ports: added SpaireLight1, SpaireLight2, SpaireLight3, SpaireLight4, SpaireLight5; removed none

Commit message: some updates
Other:
- added sheet Misc Switches (Switches.kicad_sch)
- sheet Shrimp ports: added SpaireBut1, SpaireBut2, SpaireBut3, SpaireBut4, SpaireBut5, SpaireBut6; removed none

Commit message: updated
Other:
- added sheet PSU (psu.kicad_sch)
Changed lines of the file:
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@@
+		)
+	)
+	(sheet
+		(at 39.37 63.5)
+		(size 20.32 20.32)
+		(exclude_from_sim no)
+		(in_bom yes)
+		(on_board yes)
+		(dnp no)
+		(fields_autoplaced yes)
+		(stroke
+			(width 0.1524)
+			(type solid)
+		)
+		(fill
+			(color 0 0 0 0.0000)
+		)
+		(property "Sheetname" "PSU"
+			(at 39.37 62.7884 0)
+			(effects
+				(font
+					(size 1.27 1.27)
+				)
+				(justify left bottom)
+			)
+		)
+		(property "Sheetfile" "psu.kicad_sch"
+			(at 39.37 84.4046 0)
+			(effects
+				(font
+					(size 1.27 1.27)
+				)
+				(justify left top)
+				(hide yes)
+			)
+		)
+		(instances
+			(project "BCM"
+				(path "/4f572b99-5eee-4690-a22b-0d608e2cc8a2"
+					(page "6")
+				)
+			)
 		)
 	)

Commit message: updates
Parts:
- removed J1: Conn_01x06_Socket, symbol Connector:Conn_01x06_Socket
- added J30: Power, Connector_JST:JST_XA_B06B-XASK-1_1x06_P2.50mm_Vertical, symbol Connector_Generic:Conn_01x06
Connections:
- net +BATT: now also J30.1 (Pin_1), J30.2 (Pin_2)
- net +VDC: now also J30.3 (Pin_3)
- net GND: now also J30.4 (Pin_4), J30.5 (Pin_5), J30.6 (Pin_6)
Changed lines of the file:
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@@
-	)
-	(symbol
-		(lib_id "Connector:Conn_01x06_Socket")
-		(at 30.48 30.48 0)
-		(mirror y)
-		(unit 1)
-		(exclude_from_sim no)
-		(in_bom yes)
-		(on_board yes)
-		(dnp no)
-		(fields_autoplaced yes)
-		(property "Reference" "J1"
-			(at 29.21 30.4799 0)
-			(effects
-				(font
-					(size 1.27 1.27)
-				)
-				(justify left)
-			)
-		)
-		(property "Value" "Conn_01x06_Socket"
-			(at 29.21 33.0199 0)
-			(effects
-				(font
-					(size 1.27 1.27)
-				)
-				(justify left)
-			)
-		)
-		(property "Footprint" ""
-			(at 30.48 30.48 0)
-			(effects
-				(font
-					(size 1.27 1.27)
-				)
-				(hide yes)
-			)
-		)
-		(property "Datasheet" "~"
-			(at 30.48 30.48 0)
-			(effects
-				(font
-					(size 1.27 1.27)
-				)
-				(hide yes)
-			)
-		)
-		(property "Description" "Generic connector, single row, 01x06, script generated"
-			(at 30.48 30.48 0)
-			(effects
-				(font
-					(size 1.27 1.27)
-				)
-				(hide yes)
-			)
-		)
-		(pin "1"
-		)
-		(pin "2"
-		)
-		(pin "3"
-		)
-		(pin "4"
-		)
-		(pin "6"
-		)
-		(pin "5"
-		)
-		(instances
-			(project ""
-				(path "/4f572b99-5eee-4690-a22b-0d608e2cc8a2"
-					(reference "J1")
-					(unit 1)
-				)
-			)
-		)
 	)
 	(symbol
@@
 					(unit 1)
 				)
+			)
+		)
+	)
+	(symbol
+		(lib_id "Connector_Generic:Conn_01x06")
+		(at 30.48 30.48 0)
+		(mirror y)
+		(unit 1)
+		(exclude_from_sim no)
+		(in_bom yes)
+		(on_board yes)
+		(dnp no)
+		(property "Reference" "J30"
+			(at 30.48 44.45 0)
+			(effects
+				(font
+					(size 1.27 1.27)
+				)
+			)
+		)
+		(property "Value" "Power"
+			(at 30.48 41.91 0)
+			(effects
+				(font
+					(size 1.27 1.27)
+				)
+			)
+		)
+		(property "Footprint" "Connector_JST:JST_XA_B06B-XASK-1_1x06_P2.50mm_Vertical"
+			(at 30.48 30.48 0)
+			(effects
+				(font
+					(size 1.27 1.27)
+				)
+				(hide yes)
+			)
+		)
+		(property "Datasheet" "~"
+			(at 30.48 30.48 0)
+			(effects
+				(font
+					(size 1.27 1.27)
+				)
+				(hide yes)
+			)
+		)
+		(property "Description" "Generic connector, single row, 01x06, script generated (kicad-library-utils/schlib/autogen/connector/)"
+			(at 30.48 30.48 0)
+			(effects
+				(font
+					(size 1.27 1.27)
+				)
+				(hide yes)
+			)
+		)
+		(pin "1"
+		)
+		(pin "2"
+		)
+		(pin "4"
+		)
+		(pin "5"
+		)
+		(pin "3"
+		)
+		(pin "6"
+		)
+		(instances
+			(project "BCM"
+				(path "/4f572b99-5eee-4690-a22b-0d608e2cc8a2"
+					(reference "J30")
+					(unit 1)
+				)
