File: BCM/KiCAD/psu.kicad_sch (KiCad schematic)
At the start: 20 parts, among them U1 TPS54331D

Commit message: updates
Parts:
- R81, R82, R83: footprint (none) -> Resistor_SMD:R_0805_2012Metric_Pad1.20x1.40mm_HandSolder
Connections:
- net Vin+Ve: now also D1.1 (K), D4.1 (K), F1.2; no longer C10.1, C9.1, F1.1, U1.2 (VIN)
- new net Vin+Ve (fused): C10.1, C9.1, F1.1, U1.2 (VIN)
Other:
- moved on the sheet: C10, C11, C12, C13, C14, C15, C16, C17, C9, D1, D2, D3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
