File: BCM/KiCAD/Back Button Connectors.kicad_sch (KiCad schematic)
At the start: 72 parts, among them J10 Back_9, J11 Back_10, J12 Back_11, J13 Back_12, J2 Back_1, J3 Back_2, J4 Back_3, J5 Back_4, J6 Back_5, J7 Back_6, J8 Back_7, J9 Back_8, Q1 2N7002, Q10 2N7002, Q11 2N7002, Q12 2N7002, Q2 2N7002, Q3 2N7002, Q4 2N7002, Q5 2N7002, Q6 2N7002, Q7 2N7002, Q8 2N7002, Q9 2N7002

Commit message: updated
Parts:
- added C1, C2, C3, C4: C_Small, Capacitor_SMD:C_0805_2012Metric_Pad1.18x1.45mm_HandSolder, symbol Device:C_Small
Connections:
- net +5V: now also C1.1, C2.1, C3.1, C4.1
- net GND: now also C1.2, C2.2, C3.2, C4.2

Commit message: move buttons to own supply rail
Parts:
- added C18, C19: C_Small, Capacitor_SMD:C_0805_2012Metric_Pad1.18x1.45mm_HandSolder, symbol Device:C_Small
Connections:
- net +5V: no longer R15.2, R16.2, R29.2, R30.2, R31.2, R32.2, R4.2, R45.2, R46.2, R47.2, R48.2, R8.2
- net GND: now also C18.2, C19.2
- new net Button +Ve: C18.1, C19.1, R15.2, R16.2, R29.2, R30.2, R31.2, R32.2, R4.2, R45.2, R46.2, R47.2, R48.2, R8.2
